File: EtherTenR3.brd (EAGLE design)
At the start: 68.6 x 53.3 mm, 98 parts, among them IC1 MC33269DT-5.0, IC2 APX811-44UG-7, IC3 ATMEGA16U2-MU, IC4 LM358D, IC5 ATMEGA328P TQFP32, IC6 W5100SQFP80, J1 DC_2_1MM, P1 USB-6PSMT, P2 ICSP:MAIN, P3 ICSP:USB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

Commit message: Production release R3 v2.0 files
Connections:
- net 5V: now also H2.2
Routing:
- net 5V: track 1223.4 -> 1234.7 mm
- net N$9: vias 0 -> 2
