File: EtherTenR3.sch (EAGLE design)
At the start: 98 parts, among them IC1 MC33269DT-5.0, IC2 APX811-44UG-7, IC3 ATMEGA16U2-MU, IC4 LM358D, IC5 ATMEGA328P TQFP32, IC6 W5100SQFP80, J1 DC_2_1MM, P1 USB-6PSMT, P2 ICSP:MAIN, P3 ICSP:USB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

Commit message: Improved I2C and ICSP markings; ERC and DRC for release
Connections:
- net N$3 renamed USBGND
- new net N$3: C19.1, SJ3.2
- net DTR: no longer C19.1, SJ3.2
Other:
- note added: "(Linked)"
- note added: "Freetronics EtherTen R3"
- note added: "Short across SJ1 GROUND and SJ3 RESET-EN after all other routing"
- note added: "V2.0 (2012-07-07)"
- note added: "www.freetronics.com/etherten"
- note removed: "Freetronics EtherTen (Arduino Compatible)"
- note removed: "V1.1 (2011-05-09)"
- note removed: "www.freetronics.com"
- moved on the sheet: R4, R5
Changed lines of the file:
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@@
 <circle x="238.76" y="226.06" radius="1.27" width="0.1524" layer="94"/>
 <text x="96.52" y="365.76" size="3.81" layer="94" ratio="12">Prototyping Area</text>
-<text x="7.62" y="12.7" size="2.794" layer="94">Freetronics EtherTen (Arduino Compatible)</text>
-<text x="81.28" y="6.858" size="1.778" layer="94">V1.1 (2011-05-09)</text>
-<text x="48.006" y="6.858" size="1.778" layer="94">www.freetronics.com</text>
 <text x="7.62" y="6.858" size="1.778" layer="94">SKU: ETHERTEN</text>
 <text x="33.02" y="177.8" size="1.778" layer="94">3V3 Power Supply</text>
@@
 <text x="261.62" y="96.52" size="1.778" layer="94">In Circuit Serial Programming</text>
 <text x="261.62" y="48.26" size="1.778" layer="94">micro SD Card Slot</text>
-<text x="396.24" y="12.7" size="2.794" layer="94">Freetronics EtherTen (Arduino Compatible)</text>
-<text x="469.9" y="6.858" size="1.778" layer="94">V1.1 (2011-05-09)</text>
-<text x="436.626" y="6.858" size="1.778" layer="94">www.freetronics.com</text>
-<text x="396.24" y="6.858" size="1.778" layer="94">SKU: ETHERTEN</text>
+<text x="7.62" y="12.7" size="2.794" layer="94">Freetronics EtherTen R3</text>
+<text x="81.28" y="6.858" size="1.778" layer="94">V2.0 (2012-07-07)</text>
+<text x="35.306" y="6.858" size="1.778" layer="94">www.freetronics.com/etherten</text>
 <text x="7.62" y="106.68" size="1.778" layer="94">Ethernet Module with PoE</text>
 <text x="139.7" y="149.86" size="1.778" layer="94">&lt; 4.38 Vrst, push-pull output</text>
@@
 <frame x1="0" y1="0" x2="248.92" y2="185.42" columns="8" rows="5" layer="94"/>
 <frame x1="5.08" y1="5.08" x2="109.22" y2="17.78" columns="0" rows="0" layer="94" border-left="no" border-top="no" border-right="no" border-bottom="no"/>
-<frame x1="5.08" y1="5.08" x2="43.18" y2="10.16" columns="8" rows="5" layer="94"/>
 <frame x1="78.74" y1="5.08" x2="109.22" y2="10.16" columns="8" rows="5" layer="94"/>
 <frame x1="0" y1="190.5" x2="248.92" y2="375.92" columns="8" rows="5" layer="94"/>
 <frame x1="254" y1="0" x2="502.92" y2="185.42" columns="8" rows="5" layer="94"/>
-<frame x1="393.7" y1="5.08" x2="497.84" y2="17.78" columns="0" rows="0" layer="94" border-left="no" border-top="no" border-right="no" border-bottom="no"/>
-<frame x1="393.7" y1="5.08" x2="431.8" y2="10.16" columns="8" rows="5" layer="94"/>
-<frame x1="467.36" y1="5.08" x2="497.84" y2="10.16" columns="8" rows="5" layer="94"/>
+<frame x1="5.08" y1="5.08" x2="30.48" y2="10.16" columns="8" rows="5" layer="94"/>
 <wire x1="347.98" y1="145.796" x2="347.98" y2="100.33" width="0.4064" layer="97" style="longdash"/>
 <wire x1="378.46" y1="181.356" x2="378.46" y2="146.05" width="0.4064" layer="97" style="longdash"/>
+<text x="422.275" y="112.395" size="1.27" layer="94">(Linked)</text>
+<text x="351.917" y="90.932" size="1.27" layer="94">(Linked)</text>
+<text x="358.14" y="98.298" size="1.27" layer="94">Short across SJ1 GROUND and SJ3 RESET-EN after all other routing</text>
 </plain>
 <instances>
@@
 <attribute name="VALUE" x="422.148" y="140.335" size="1.778" layer="96"/>
 </instance>
-<instance part="R4" gate="G$1" x="419.1" y="121.92" smashed="yes" rot="R180">
-<attribute name="NAME" x="422.148" y="122.1486" size="1.778" layer="95"/>
+<instance part="R4" gate="G$1" x="416.56" y="121.92" smashed="yes" rot="R180">
+<attribute name="NAME" x="419.608" y="122.1486" size="1.778" layer="95"/>
 <attribute name="VALUE" x="405.13" y="116.078" size="1.778" layer="96"/>
 </instance>
-<instance part="R5" gate="G$1" x="419.1" y="119.38" smashed="yes" rot="R180">
-<attribute name="NAME" x="422.148" y="119.6086" size="1.778" layer="95"/>
+<instance part="R5" gate="G$1" x="416.56" y="119.38" smashed="yes" rot="R180">
+<attribute name="NAME" x="419.608" y="119.6086" size="1.778" layer="95"/>
 <attribute name="VALUE" x="405.13" y="113.538" size="1.778" layer="96"/>
 </instance>
@@
 <junction x="431.8" y="104.14"/>
 <pinref part="GND39" gate="1" pin="GND"/>
+<pinref part="SJ1" gate="1" pin="2"/>
 <wire x1="421.64" y1="104.14" x2="424.18" y2="104.14" width="0.1524" layer="91"/>
-<pinref part="SJ1" gate="1" pin="2"/>
 <wire x1="424.18" y1="104.14" x2="431.8" y2="104.14" width="0.1524" layer="91"/>
 <wire x1="424.18" y1="104.14" x2="424.18" y2="111.76" width="0.1524" layer="91"/>
@@
 <wire x1="477.52" y1="96.52" x2="477.52" y2="129.54" width="0.1524" layer="91"/>
 <wire x1="477.52" y1="129.54" x2="474.98" y2="129.54" width="0.1524" layer="91"/>
-<wire x1="370.84" y1="86.36" x2="360.68" y2="86.36" width="0.1524" layer="91"/>
-<wire x1="360.68" y1="91.44" x2="360.68" y2="86.36" width="0.1524" layer="91"/>
-<wire x1="350.52" y1="91.44" x2="360.68" y2="91.44" width="0.1524" layer="91"/>
 <junction x="350.52" y="86.36"/>
 <junction x="347.98" y="86.36"/>
-<junction x="360.68" y="86.36"/>
 <label x="347.98" y="96.52" size="1.778" layer="95"/>
 <pinref part="SJ3" gate="1" pin="1"/>
 <pinref part="SJ2" gate="1" pin="2"/>
 <pinref part="IC3" gate="G$1" pin="(CTS)PD7"/>
-<pinref part="C19" gate="G$1" pin="1"/>
-<pinref part="SJ3" gate="1" pin="2"/>
 </segment>
 </net>
@@
 <net name="RD-" class="0">
 <segment>
-<wire x1="424.18" y1="121.92" x2="434.34" y2="121.92" width="0.1524" layer="91"/>
+<wire x1="421.64" y1="121.92" x2="434.34" y2="121.92" width="0.1524" layer="91"/>
 <label x="429.26" y="121.92" size="1.778" layer="95"/>
 <pinref part="R4" gate="G$1" pin="1"/>
@@
 <net name="RD+" class="0">
 <segment>
-<wire x1="424.18" y1="119.38" x2="434.34" y2="119.38" width="0.1524" layer="91"/>
+<wire x1="421.64" y1="119.38" x2="434.34" y2="119.38" width="0.1524" layer="91"/>
 <label x="429.26" y="119.38" size="1.778" layer="95"/>
 <pinref part="R5" gate="G$1" pin="1"/>
@@
 <wire x1="396.24" y1="127" x2="406.4" y2="127" width="0.1524" layer="91"/>
 <wire x1="406.4" y1="127" x2="406.4" y2="119.38" width="0.1524" layer="91"/>
-<wire x1="406.4" y1="119.38" x2="414.02" y2="119.38" width="0.1524" layer="91"/>
+<wire x1="406.4" y1="119.38" x2="411.48" y2="119.38" width="0.1524" layer="91"/>
 <junction x="396.24" y="127"/>
 <pinref part="Z1" gate="G$1" pin="1"/>
@@
 <wire x1="398.78" y1="119.38" x2="398.78" y2="129.54" width="0.1524" layer="91"/>
 <wire x1="398.78" y1="129.54" x2="381" y2="129.54" width="0.1524" layer="91"/>
-<wire x1="414.02" y1="121.92" x2="408.94" y2="121.92" width="0.1524" layer="91"/>
+<wire x1="411.48" y1="121.92" x2="408.94" y2="121.92" width="0.1524" layer="91"/>
 <wire x1="408.94" y1="121.92" x2="408.94" y2="129.54" width="0.1524" layer="91"/>
 <wire x1="408.94" y1="129.54" x2="398.78" y2="129.54" width="0.1524" layer="91"/>
@@
 </net>
 <net name="N$3" class="0">
+<segment>
+<pinref part="C19" gate="G$1" pin="1"/>
+<wire x1="370.84" y1="86.36" x2="360.68" y2="86.36" width="0.1524" layer="91"/>
+<wire x1="360.68" y1="91.44" x2="360.68" y2="86.36" width="0.1524" layer="91"/>
+<junction x="360.68" y="86.36"/>
+<pinref part="SJ3" gate="1" pin="2"/>
+</segment>
+</net>
+<net name="USBGND" class="0">
 <segment>
 <wire x1="434.34" y1="116.84" x2="424.18" y2="116.84" width="0.1524" layer="91"/>
@@
 <wire x1="424.18" y1="116.84" x2="424.18" y2="114.3" width="0.1524" layer="91"/>
 <junction x="424.18" y="116.84"/>
+<label x="421.64" y="116.84" size="1.778" layer="95"/>
 </segment>
 </net>
@@
 </sheet>
 </sheets>
+<errors>
+</errors>
 </schematic>
 </drawing>

Commit message: Production release R3 v2.0 files
Connections:
- net 5V: now also H2.2
Other:
- note added: "IOREF"
- moved on the sheet: C1
Changed lines of the file:
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@@
 <text x="33.02" y="177.8" size="1.778" layer="94">3V3 Power Supply</text>
 <text x="195.58" y="177.8" size="1.778" layer="94">Status Display</text>
-<text x="10.16" y="215.9" size="2.1844" layer="94" ratio="10" rot="R90">Headers / Solder Pads</text>
+<text x="10.16" y="218.44" size="2.1844" layer="94" ratio="10" rot="R90">Headers / Solder Pads</text>
 <text x="40.132" y="156.464" size="1.6764" layer="94">Dual Footprint</text>
 <text x="95.25" y="177.8" size="1.778" layer="94">1.8V / 3.3V Decoupling</text>
 <text x="91.44" y="200.66" size="2.54" layer="94" ratio="10">Draw your project schematic here</text>
-<text x="242.57" y="215.9" size="2.1844" layer="94" ratio="10" rot="R90">Headers / Solder Pads</text>
+<text x="244.348" y="223.774" size="2.1844" layer="94" ratio="10" rot="R90">Headers / Solder Pads</text>
 <text x="236.22" y="276.86" size="1.6764" layer="94" ratio="12" rot="R90">D10, 11, 12, 13 used by Ethernet interface.</text>
 <text x="238.76" y="276.86" size="1.6764" layer="94" ratio="12" rot="R90">D2 used if Wiznet Ethernet IC "interrupt" jumper enabled.</text>
@@
 <text x="351.917" y="90.932" size="1.27" layer="94">(Linked)</text>
 <text x="358.14" y="98.298" size="1.27" layer="94">Short across SJ1 GROUND and SJ3 RESET-EN after all other routing</text>
+<text x="27.94" y="256.54" size="1.778" layer="94">IOREF</text>
 </plain>
 <instances>
 <instance part="H3" gate="G$1" x="17.78" y="223.52" rot="MR180"/>
 <instance part="H4" gate="G$1" x="231.14" y="223.52" smashed="yes" rot="MR0">
+<attribute name="VALUE" x="240.284" y="237.236" size="1.778" layer="96" rot="MR0"/>
 <attribute name="NAME" x="233.172" y="210.82" size="1.778" layer="95" rot="MR0"/>
 </instance>
@@
 <attribute name="VALUE" x="325.12" y="137.16" size="1.778" layer="96"/>
 </instance>
-<instance part="C1" gate="G$1" x="231.14" y="284.48" smashed="yes">
-<attribute name="NAME" x="225.679" y="280.924" size="1.778" layer="95" rot="R90"/>
-<attribute name="VALUE" x="228.219" y="278.384" size="1.778" layer="96" rot="R90"/>
-</instance>
-<instance part="GND50" gate="1" x="231.14" y="276.86"/>
+<instance part="C1" gate="G$1" x="231.14" y="287.02" smashed="yes">
+<attribute name="NAME" x="225.679" y="283.464" size="1.778" layer="95" rot="R90"/>
+<attribute name="VALUE" x="228.219" y="280.924" size="1.778" layer="96" rot="R90"/>
+</instance>
+<instance part="GND50" gate="1" x="231.14" y="279.4"/>
 <instance part="RN8" gate="A" x="297.18" y="17.78" rot="R90"/>
 <instance part="RN8" gate="B" x="287.02" y="17.78" rot="R90"/>
@@
 <instance part="FID3" gate="G$1" x="241.3" y="20.32"/>
 <instance part="H2" gate="G$1" x="17.78" y="251.46" rot="MR180"/>
-<instance part="H1" gate="G$1" x="236.22" y="264.16" rot="MR0"/>
+<instance part="H1" gate="G$1" x="236.22" y="264.16" smashed="yes" rot="MR0">
+<attribute name="VALUE" x="241.808" y="272.542" size="1.778" layer="96" rot="MR0"/>
+<attribute name="NAME" x="233.426" y="241.3" size="1.778" layer="95" rot="MR0"/>
+</instance>
 <instance part="P1" gate="G$1" x="375.92" y="127" smashed="yes" rot="R180">
 <attribute name="NAME" x="375.92" y="125.73" size="2.54" layer="95" rot="R90"/>
@@
 <segment>
 <pinref part="H1" gate="G$1" pin="10"/>
-<wire x1="226.06" y1="269.24" x2="210.82" y2="269.24" width="0.2032" layer="91"/>
+<wire x1="226.06" y1="269.24" x2="210.82" y2="269.24" width="0.1524" layer="91"/>
 <label x="210.82" y="269.24" size="1.778" layer="95"/>
 </segment>
@@
 </segment>
 <segment>
-<wire x1="231.14" y1="279.4" x2="231.14" y2="281.94" width="0.1524" layer="91"/>
 <pinref part="GND50" gate="1" pin="GND"/>
 <pinref part="C1" gate="G$1" pin="2"/>
+<wire x1="231.14" y1="284.48" x2="231.14" y2="281.94" width="0.1524" layer="91"/>
 </segment>
 <segment>
@@
 <wire x1="210.82" y1="264.16" x2="218.44" y2="264.16" width="0.1524" layer="91"/>
 <wire x1="218.44" y1="264.16" x2="226.06" y2="264.16" width="0.1524" layer="91"/>
-<wire x1="218.44" y1="264.16" x2="218.44" y2="292.1" width="0.1524" layer="91"/>
-<wire x1="231.14" y1="289.56" x2="231.14" y2="292.1" width="0.1524" layer="91"/>
-<wire x1="218.44" y1="292.1" x2="231.14" y2="292.1" width="0.1524" layer="91"/>
+<wire x1="218.44" y1="264.16" x2="218.44" y2="297.18" width="0.1524" layer="91"/>
+<wire x1="231.14" y1="292.1" x2="231.14" y2="297.18" width="0.1524" layer="91"/>
+<wire x1="218.44" y1="297.18" x2="231.14" y2="297.18" width="0.1524" layer="91"/>
 <junction x="218.44" y="264.16"/>
 <label x="210.82" y="264.16" size="1.778" layer="95"/>
@@
 <pinref part="U$11" gate="G$1" pin="5V"/>
 <pinref part="RN4" gate="A" pin="2"/>
+</segment>
+<segment>
+<pinref part="H2" gate="G$1" pin="2"/>
+<wire x1="22.86" y1="256.54" x2="35.56" y2="256.54" width="0.1524" layer="91"/>
+<label x="22.86" y="256.54" size="1.778" layer="95"/>
 </segment>
 </net>
@@
 <segment>
 <pinref part="H1" gate="G$1" pin="9"/>
-<wire x1="226.06" y1="266.7" x2="210.82" y2="266.7" width="0.2032" layer="91"/>
+<wire x1="226.06" y1="266.7" x2="210.82" y2="266.7" width="0.1524" layer="91"/>
 <label x="210.82" y="266.7" size="1.778" layer="95"/>
 </segment>
