File: EtherTen.sch (EAGLE design)
At the start: 98 parts, among them IC1 MC33269DT-5.0, IC2 APX811-44UG-7, IC3 ATMEGA16U2-MU, IC4 LM358D, IC5 ATMEGA328P TQFP32, IC6 W5100SQFP80, J1 DC_2_1MM, P1 USB-6PSMT, P2 ICSP:MAIN, P3 ICSP:USB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

Commit message: Added I2C MAC ROM in preparation for v3.0
Parts:
- added IC7: MCP24AA025E48, freetronics-jon:MCP24AA025E48
- added R14, R15: 4K7, freetronics-master-v1.1:RESISTOR0603
- added SJ5, SJ6: SJCN, freetronics-jon:SJCN
Connections:
- new net N$29: IC7.SDA, R14.2, SJ5.2
- new net N$5: IC7.SCL, R15.2, SJ6.2
- net 5V: now also IC7.VCC, R14.1, R15.1; no longer H2.2
- net A4_SDA: now also SJ5.1
- net A5_SCL: now also SJ6.1
- net GND: now also IC7.A0, IC7.A1, IC7.GND
Other:
- note added: "Freetronics EtherTen"
- note added: "I2C Addr: 70 (0x50)"
- note added: "SKU: ET"
- note added: "V3.0 (2013-09-06)"
- note added: "www.freetronics.com/et"
- note removed: "Freetronics EtherTen R3"
- note removed: "IOREF"
- note removed: "SKU: ETHERTEN"
- note removed: "V2.0 (2012-07-07)"
- note removed: "www.freetronics.com/etherten"
- moved on the sheet: C1, C27, RN7A, RN7C, RN8D
